Commit message: various

File: src/robotino_description/urdf/robotino_body.urdf.xacro (robot description, xacro)
@@ -1,19 +1,32 @@
 <?xml version="1.0"?>
 <robot xmlns:xacro="http://wiki.ros.org/xacro">
-    <xacro:property name="M_PI" value="3.14159"/>
     <xacro:property name="M_SCALE" value="0.01"/>
     <xacro:property name="BASE_RADIUS" value="0.18"/>
-    <xacro:property name="BASE_HEIGHT" value="0.05"/>
-    <xacro:property name="BASE_MASS" value="20"/>
+    <xacro:property name="BASE_HEIGHT" value="0.03"/>
+    <xacro:property name="BASE_MASS" value="20"/> <!-- 20 -->
+    <xacro:property name="M_PI" value="3.1415926535897931"/>
+    <xacro:property name="width" value="0.5"/> <!-- Square dimensions (widthxwidth) of beams -->
+    <xacro:property name="height" value="0.5"/> <!-- Link 1 -->
+    <xacro:property name="width_2" value="0.1"/> <!-- Square dimensions (widthxwidth) of beams -->
+    <xacro:property name="height_2" value="0.5"/> <!-- Link 1 -->
+    <xacro:property name="axel_offset" value="0.05"/> <!-- Space btw top of beam and the each joint -->
+    <xacro:property name="roll" value="${M_PI/2}"/> <!-- Space btw top of beam and the each joint -->
+    <xacro:property name="yaw" value="${M_PI/2}"/> <!-- Space btw top of beam and the each joint -->
     <!-- robotino_body -->
     <xacro:macro name="robotino_body">
         <!-- base_link -->
-        <link name="base_link">
+        <link name="base_link"/>
+        <joint name="base_body_joint" type="fixed">
+            <parent link="base_link"/>
+            <child link="base_body_link"/>
+            <origin xyz="0 0 0" rpy="0 0 3.1415"/>
+        </joint>
+        <link name="base_body_link">
             <inertial>
-                <mass value="${BASE_MASS}" />
-                <origin xyz="0 0 0" />
-                <inertia ixx="1.0" ixy="0.0" ixz="0.0"
-                    iyy="1.0" iyz="0.0"
-                    izz="1.0" />
+                <mass value="${BASE_MASS}"/>
+                <origin xyz="0 0 0.035" rpy="0 0 3.1415"/>
+                <inertia ixx="0.8750" ixy="0.0" ixz="0.0"
+                         iyy="0.875" iyz="0.0"
+                         izz="1"/>
             </inertial>
             <visual>
@@ -21,39 +34,36 @@
                 <geometry>
                     <mesh filename="package://robotino_description/meshes/parts/robotino_base.dae"
-                        scale="${M_SCALE} ${M_SCALE} ${M_SCALE}"/>
+                          scale="${M_SCALE} ${M_SCALE} ${M_SCALE}"/>
                 </geometry>
             </visual>
             <collision>
-                <origin xyz="0 0 ${BASE_HEIGHT/2}" rpy="0 0 0" />
+                <origin xyz="0 0 0" rpy="0 0 ${M_PI/2}"/>
                 <geometry>
-                    <cylinder radius="${BASE_RADIUS}" length="${BASE_HEIGHT}"/>
+                    <mesh filename="package://robotino_description/meshes/parts/robotino_base.stl"
+                          scale="${M_SCALE} ${M_SCALE} ${M_SCALE}"/>
                 </geometry>
             </collision>
         </link>
-        <gazebo reference="base_link">
-            <material>Gazebo/White</material>
-            <turnGravityOff>false</turnGravityOff>
-        </gazebo>
         <!-- wheels -->
-        <wheel name="wheel0" parent="base_link">
-            <origin xyz="0.065 0.11 0.04" rpy="0 0 ${M_PI/3}"/>
-            <axis xyz="-1 0 0"/>
-        </wheel>
-        <wheel name="wheel1" parent="base_link">
-            <origin xyz="-0.13 0 0.04" rpy="0 0 0"/>
-            <axis xyz="1 0 0"/>
-        </wheel>
-        <wheel name="wheel2" parent="base_link">
-            <origin xyz="0.065 -0.11 0.04" rpy="0 0 -${M_PI/3}"/>
-            <axis xyz="-1 0 0"/>
-        </wheel>
+        <xacro:wheel name="wheel2" parent="base_link">
+            <origin xyz="-0.0001 0.1825 0.059154" rpy="0 0 0"/>
+    	    <axis xyz="0 1 0" rpy="0 0 0"/>
+        </xacro:wheel>
+        <xacro:wheel name="wheel0" parent="base_link">
+            <origin xyz="-0.157067 -0.090625 0.059154" rpy="0 0 2.094395102393195"/>
+    	    <axis xyz="0 1 0" rpy="0 0 0"/>
+        </xacro:wheel>
+        <xacro:wheel name="wheel1" parent="base_link">
+            <origin xyz="0.156867 -0.090625 0.059154" rpy="0 0 -2.094395102393195"/>
+   	    <axis xyz="0 1 0" rpy="0 0 0"/>
+        </xacro:wheel>
         <!-- others -->
         <!-- lasersensor -->
- 	    <lasersensor name="lasersensor" parent="base_link">
+        <xacro:lasersensor name="lasersensor" parent="base_link">
             <origin xyz="0.0 0 0.26" rpy="0 0 0"/>
-        </lasersensor>
+        </xacro:lasersensor>
         <!-- pantilt holder part 1-->
         <xacro:pantilt name="pantilt" parent="base_link">
-            <origin xyz="0.0 0 0.33" rpy="0 0 0.5"/>
+            <origin xyz="0.0 0 0.325" rpy="0 0 0"/>
         </xacro:pantilt>
         <!-- pantilt holder part 2-->
@@ -65,63 +75,8 @@
             <origin xyz="0.0 0 0" rpy="0 0 0"/>
         </xacro:cameraholder>
-        <!-- gazebo control -->
-        <!--
-        <gazebo reference="lasersensor_link">
-            <sensor type="ray" name="head_hokuyo_sensor">
-                <pose>0 0 0 0 0 0</pose>
-                <visualize>true</visualize>
-                <update_rate>20</update_rate>
-                <ray>
-                    <scan>
-                        <horizontal>
-                            <samples>300</samples>
-                            <resolution>1</resolution>
-                            <min_angle>-3.14159</min_angle>
-                            <max_angle>+3.14159</max_angle>
-                        </horizontal>
-                    </scan>
-                    <range>
-                        <min>0.10</min>
-                        <max>12.0</max>
-                        <resolution>0.01</resolution>
-                    </range>
-                    <noise>
-                        <type>gaussian</type>
-                        <mean>0.0</mean>
-                        <stddev>0.01</stddev>
-                    </noise>
-                    </ray>
-                    <plugin name="gazebo_ros_head_hokuyo_controller" filename="libgazebo_ros_laser.so">
-                        <topicName>robot/laser/scan</topicName>
-                        <robotNamespace>/</robotNamespace>
-                        <frameName>lasersensor_link</frameName>
-                    </plugin>
-            </sensor>
-        </gazebo>
-        <gazebo>
-            <plugin name="object_controller" filename="libgazebo_ros_planar_move.so">
-                <commandTopic>cmd_vel</commandTopic>
-                <odometryTopic>odom</odometryTopic>
-                <odometryFrame>odom</odometryFrame>
-                <odometryRate>20</odometryRate>
-                <robotBaseFrame>base_link</robotBaseFrame>
-            </plugin>
-        </gazebo>
-        <gazebo>
-            <plugin name="gazebo_ros_control" filename="libgazebo_ros_control.so">
-             <robotNamespace>/rrbot</robotNamespace>
-            </plugin>
-        </gazebo>
-        <gazebo>
-            <plugin name="object_controller2" filename="libgazebo_ros_planar_move.so">
-                <commandTopic>camera/cmd_vel</commandTopic>
-                <odometryTopic>base_link</odometryTopic>
-                <odometryFrame>base_link</odometryFrame>
-                <odometryRate>20</odometryRate>
-                <robotBaseFrame>cameraholder_link</robotBaseFrame>
-            </plugin>
-            <plugin name="gazebo_ros_control" filename="libgazebo_ros_control.so"/>
-        </gazebo>
-         -->
+        <!-- imu -->
+        <xacro:imu name="imu" parent="base_link">
+            <origin xyz="0.0 0 10" rpy="0 3.1415 0"/>
+        </xacro:imu>
     </xacro:macro>
 </robot>

File: src/robotino_description/urdf/robotino_parts.urdf.xacro (robot description, xacro)
@@ -9,35 +9,28 @@
         <link name="${name}_link">
             <inertial>
-                <mass value="0.00001"/>
-                <origin xyz="0 0 0"/>
-                <inertia ixx="1.0" ixy="0.0" ixz="0.0" iyy="1.0" iyz="0.0" izz="1.0"/>
-            </inertial>
-            <visual>
+                <mass value="2"/>
                 <origin xyz="0 0 0" rpy="0 0 0"/>
-                <geometry>
-                    <mesh filename="package://robotino_description/meshes/parts/robotino_wheel.dae" scale="${M_SCALE} ${M_SCALE} ${M_SCALE}"/>
-                </geometry>
-            </visual>
-        </link>
-        <gazebo reference="${name}_link">
-            <material>Gazebo/Yellow</material>
-            <turnGravityOff>false</turnGravityOff>
-        </gazebo>
+                <inertia ixx="0.04" ixy="0.0" ixz="0.0" iyy="0.04" iyz="0.0" izz="0.04"/>
+            </inertial>
+            <visual>
+                <origin xyz="0 0 0" rpy="0 0 0"/>
+                <geometry>
+                    <mesh filename="package://robotino_description/meshes/parts/robotino_wheel.dae"
+                          scale="${M_SCALE} ${M_SCALE} ${M_SCALE}"/>
+                </geometry>
+            </visual>
+            <collision>
+                <origin xyz="0 0 0" rpy="0 ${M_PI/2} 0"/>
+                <geometry>
+                    <cylinder length="0.04" radius="0.04"/>
+                </geometry>
+            </collision>
+        </link>
         <joint name="${name}_joint" type="continuous">
-            <xacro:insert_block name="origin" />
+            <xacro:insert_block name="origin"/>
             <xacro:insert_block name="axis"/>
             <parent link="${parent}"/>
             <child link="${name}_link"/>
         </joint>
-        <transmission name="${name}_joint_trans">
-            <type>transmission_interface/SimpleTransmission</type>
-            <joint name="${name}_joint">
-                <hardwareInterface>hardware_interface/EffortJointInterface</hardwareInterface>
-            </joint>
-            <actuator name="${name}_motor">
-                <hardwareInterface>hardware_interface/EffortJointInterface</hardwareInterface>
-                <mechanicalReducation>1</mechanicalReducation>
-            </actuator>
-        </transmission>
     </xacro:macro>
     <!-- laser sensor-->
@@ -49,5 +42,5 @@
                 rpy="0 0 0" />
             <mass
-                value="0.15915" />
+                value="0.015915" />
             <inertia
                 ixx="7.2795244626149E-05"
@@ -75,8 +68,4 @@
             </collision>
         </link>
-        <gazebo reference="${name}_link">
-            <material>Gazebo/Black</material>
-            <turnGravityOff>false</turnGravityOff>
-        </gazebo>
         <joint name="${name}_joint" type="fixed">
             <xacro:insert_block name="origin"/>
@@ -88,22 +77,22 @@
     <xacro:macro name="pantilt" params="parent name *origin">
         <link name="${name}_link">
-            <inertial>
-            <origin
-                xyz="-0.00076068 0.053384 -0.00086946"
-                rpy="0 0 0" />
-            <mass
-                value="1.7709" />
-            <inertia
-                ixx="0.022066"
-                ixy="0.00017957"
-                ixz="-1.0212E-05"
-                iyy="0.016545"
-                iyz="0.00019743"
-                izz="0.022127" />
-            </inertial>
-            <visual>
-                <origin xyz="0 0 0" rpy="0 0 0" />
-                <geometry>
-                    <mesh filename="package://robotino_description/pantiltholder/meshes/camerabase_link.STL" />
+        <inertial>
+        <origin
+            xyz="-0.00076068 0.053384 -0.00086946"
+            rpy="0 0 0" />
+        <mass
+            value="0.17709" />
+        <inertia
+            ixx="0.022066"
+            ixy="0.00017957"
+            ixz="-1.0212E-05"
+            iyy="0.016545"
+            iyz="0.00019743"
+            izz="0.022127" />
+        </inertial>
+            <visual>
+                <origin xyz="0 0 0" rpy="0 0 0" />
+                <geometry>
+                    <mesh filename="package://robotino_description/pantiltholder/meshes/camerabase_Link.STL" />
                 </geometry>
                 <material
@@ -115,11 +104,8 @@
                 <origin xyz="0 0 0" rpy="0 0 0" />
                 <geometry>
-                    <mesh filename="package://robotino_description/pantiltholder/meshes/camerabase_link.STL" />
-                </geometry>
-            </collision>
-        </link>
-        <gazebo reference="${name}_link">
-            <turnGravityOff>false</turnGravityOff>
-        </gazebo>
+                    <mesh filename="package://robotino_description/pantiltholder/meshes/camerabase_Link.STL" />
+                </geometry>
+            </collision>
+        </link>
         <joint name="${name}_joint" type="fixed">
             <xacro:insert_block name="origin"/>
@@ -162,7 +148,4 @@
             </collision>
         </link>
-        <gazebo reference="${name}_link">
-            <turnGravityOff>false</turnGravityOff>
-        </gazebo>
         <joint name="${name}_joint" type="fixed">
             <xacro:insert_block name="origin"/>
@@ -174,20 +157,20 @@
     <xacro:macro name="cameraholder" params="parent name *origin">
         <link name="${name}_link">
-            <inertial>
-            <origin
-                xyz="0.08119 -9.6149E-11 -0.006335"
-                rpy="0 0 0" />
-            <mass
-                value="0.061321" />
-            <inertia
-                ixx="1.6538E-06"
-                ixy="1.156E-14"
-                ixz="1.0178E-05"
-                iyy="7.7966E-05"
-                iyz="-6.9072E-14"
-                izz="7.6312E-05" />
-            </inertial>
-            <visual>
-                <origin xyz="0 0 0.1785" rpy="0.050256 -1.5708 0" />
+        <inertial>
+        <origin
+            xyz="0.08119 -9.6149E-11 -0.006335"
+            rpy="0 0 0" />
+        <mass
+            value="0.061321" />
+        <inertia
+            ixx="1.6538E-06"
+            ixy="1.156E-14"
+            ixz="1.0178E-02"
+            iyy="7.7966E-05"
+            iyz="-6.9072E-14"
+            izz="7.6312E-02" />
+        </inertial>
+            <visual>
+                <origin xyz="0 0 0" rpy="0 0 0" />
                 <geometry>
                     <mesh filename="package://robotino_description/pantiltholder/meshes/cameraholder_Link.STL" />
@@ -199,5 +182,5 @@
             </visual>
             <collision>
-                <origin xyz="0 0 0.1785" rpy="0 -1.5708 0" />
+                <origin xyz="0 0 0" rpy="0 0 0" />
             <geometry>
                 <mesh filename="package://robotino_description/pantiltholder/meshes/cameraholder_Link.STL" />
@@ -208,5 +191,5 @@
             <xacro:insert_block name="origin"/>
             <origin
-                xyz="0 0 0.1785"
+                xyz="0 0 0"
                 rpy="0.050256 -1.5708 0" />
             <parent link="${parent}"/>
@@ -214,14 +197,36 @@
             <axis xyz="0 0 1" />
         </joint>
-        <transmission name="${name}_joint_trans">
-            <type>transmission_interface/SimpleTransmission</type>
-            <joint name="${name}_joint">
-                <hardwareInterface>hardware_interface/PositionJointInterface</hardwareInterface>
-            </joint>
-            <actuator name="${name}_motor">
-                <hardwareInterface>hardware_interface/PositionJointInterface</hardwareInterface>
-                <mechanicalReducation>1</mechanicalReducation>
-            </actuator>
-        </transmission>
+    </xacro:macro>
+    <!-- imu -->
+    <xacro:macro name="imu" params="parent name *origin">
+        <link name="imu_link">
+            <visual>
+                <origin xyz="0 0 -10" rpy="0 ${M_PI} 0"/>
+                <geometry>
+                    <box size="0.018 0.016 0.007"/>
+                </geometry>
+                <material name="xsens-orange"/>
+            </visual>
+            <collision>
+                <origin xyz="0 0 0" rpy="0 ${M_PI} 0"/>
+                <geometry>
+                    <box size="0.057 0.041 0.024"/>
+                </geometry>
+            </collision>
+            <inertial>
+                <mass value="0"/>
+                <origin xyz="0 0 0"/>
+                <inertia ixx="1.60333333333e-05" ixy="0.0" ixz="0.0" iyy="2.80333333333e-05" iyz="0.0"
+                         izz="1.60333333333e-05"/>
+            </inertial>
+        </link>
+        <joint name="${parent}_to_imu_link" type="fixed">
+            <parent link="${parent}"/>
+            <child link="imu_link"/>
+            <origin xyz="0 0 0" rpy="${M_PI} 0 0"/>
+        </joint>
+        <material name="xsens-orange">
+            <color rgba="0.8862745098 0.56862745098 0.09019607843 1"/>
+        </material>
     </xacro:macro>
 </robot>
