Commit message: edits to urdf

File: src/robotino_description/urdf/robotino.urdf.xacro (robot description, xacro)
@@ -8,5 +8,5 @@
     <xacro:sensor_d435
         parent="cameraholder_link">
-        <origin xyz="0 0 0.32" rpy="0 0 0"/>
+        <origin xyz="0.0235 -0.022 0.32" rpy="3.141592 0 0"/>
     </xacro:sensor_d435>
 </robot>

File: src/robotino_description/urdf/robotino_parts.urdf.xacro (robot description, xacro)
@@ -192,5 +192,5 @@
             <origin
                 xyz="0 0 0"
-                rpy="0.050256 -1.5708 0" />
+                rpy="0.0 -1.5708 0" />
             <parent link="${parent}"/>
             <child link="${name}_link"/>
