Commit message: updating -- probably working

File: src/robotino_description/urdf/robotino_sim.urdf (robot description, URDF)
Before this commit: robot robotino, 23 links, 22 joints
Links:
- removed link base_body_link
- removed link camera_bottom_screw_frame
- removed link camera_color_frame
- removed link camera_color_optical_frame
- removed link camera_depth_frame
- removed link camera_depth_optical_frame
- removed link camera_left_ir_frame
- removed link camera_left_ir_optical_frame
- removed link camera_link
- removed link camera_right_ir_frame
- removed link camera_right_ir_optical_frame
- removed link int_link_xy
- removed link int_link_yw
- removed link world
- link base_link: mass None -> 0.5; geometry collision box size=0 0 0; visual mesh filename=package://robotino_description/meshes/parts/robotino_base.d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 scale=0.01 0.01 0.01
- link cameraholder_link: geometry visual mesh filename=package://robotino_description/pantiltholder/meshes/camerah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
- link imu_link: geometry visual box size=0.018 0.016 0.007
- link lasersensor_link: geometry visual mesh filename=package://robotino_description/lidar/meshes/lidar.STL
- link pantilt_link: geometry visual mesh filename=package://robotino_description/pantiltholder/meshes/camerab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
- link pantiltring_link: geometry visual mesh filename=package://robotino_description/ring/meshes/ring.STL
- link wheel0_link: geometry visual mesh filename=package://robotino_description/meshes/parts/robotino_wheel.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 scale=0.01 0.01 0.01
- link wheel1_link: geometry visual mesh filename=package://robotino_description/meshes/parts/robotino_wheel.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 scale=0.01 0.01 0.01
- link wheel2_link: geometry visual mesh filename=package://robotino_description/meshes/parts/robotino_wheel.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 scale=0.01 0.01 0.01
Joints:
- removed joint base_body_joint
- removed joint camera_color_joint
- removed joint camera_color_optical_joint
- removed joint camera_depth_joint
- removed joint camera_depth_optical_joint
- removed joint camera_joint
- removed joint camera_left_ir_joint
- removed joint camera_left_ir_optical_joint
- removed joint camera_link_joint
- removed joint camera_right_ir_joint
- removed joint camera_right_ir_optical_joint
- removed joint joint_x
- removed joint joint_y
- removed joint revolute_w
- joint lasersensor_joint: parent base_link -> yaw_link
- joint pantilt_joint: origin xyz=0.0 0 0.33 rpy=0 0 0 -> xyz=0.0 0 0.157 rpy=0 0 0; parent base_link -> pantiltring_link
- joint pantiltring_joint: parent base_link -> yaw_link
